File: Lipo Discharger.kicad_pcb (KiCad board)
At the start: 2 copper layers, 137 x 99.5 mm, 99 parts, among them J1 Conn_01x04_Male, J11 Conn_01x04_Male, J2 USB_C_Receptacle_USB2.0_16P, J3 Conn_01x04_Male, J4 XT60_P1, J5 XT60_P1, J6 XT60_P1, J7 XT60_P1, J8 XT60_P1, J9 FAN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

Commit message: V0.2.0 after sending to manufacturing
Parts:
- moved SW1 2.70 mm to (89.2, 121.8)
- moved J2 1.94 mm to (103.5, 121.0)
- moved R54 1.58 mm to (139.5, 113.0), turned to -90 degrees
- moved RP_SCL1 0.74 mm to (129.2, 115.0)
- moved RP_SDA1 0.74 mm to (131.7, 115.0)
- moved D13 0.50 mm to (147.1, 108.5)
- moved R2 0.47 mm to (99.0, 112.0)
- moved C11 0.34 mm to (39.3, 124.0)
- moved J4 0.31 mm to (31.0, 33.6)
- moved J6 0.31 mm to (83.1, 33.6)
- moved J8 0.31 mm to (135.1, 33.6)
- moved J5 0.31 mm to (57.1, 33.6)
- moved J7 0.31 mm to (109.1, 33.6)
- renumbered J9 to FAN, J3 to I2C, J11 to ST-Link, J1 to UART
Routing:
- net GND: track 0.00 -> 571.4 mm, vias 0 -> 6
- net +BATT: track 0.00 -> 187.5 mm, vias 0 -> 2
- net +3.3V: track 0.00 -> 183.8 mm, vias 0 -> 1
- net ADC_P5: track 0.00 -> 179.2 mm, vias 0 -> 2
- net ADC_P4: track 0.00 -> 170.5 mm, vias 0 -> 2
- net GATE_P5: track 0.00 -> 149.7 mm, vias 0 -> 2
- net +5V: track 0.00 -> 139.1 mm, vias 0 -> 1
- net ADC_P3: track 0.00 -> 127.8 mm, vias 0 -> 2
- net GATE_P4: track 0.00 -> 120.5 mm, vias 0 -> 2
- net /STM32/SWDIO: track 0.00 -> 113.4 mm
- net /STM32/SWCLK: track 0.00 -> 113.4 mm
- net /STM32/USART1_TX: track 0.00 -> 112.8 mm, vias 0 -> 1
- net /STM32/USART1_RX: track 0.00 -> 111.9 mm, vias 0 -> 1
- net FAN_CTRL: track 0.00 -> 110.9 mm, vias 0 -> 2
- net /STM32/I2C2_SCL: track 0.00 -> 106.6 mm, vias 0 -> 3
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Other:
- board size 137 x 99.5 mm -> 137 x 100 mm
