File: Lipo Discharger.kicad_sch (KiCad schematic)
At the start: 15 parts, among them U1 MP2359DJ-LF-Z, U2 AMS1117-3.3

Commit message: Complete board redesign
Parts:
- removed C7, C8: 100nF, Capacitor_SMD:C_0805_2012Metric_Pad1.18x1.45mm_HandSolder, symbol Device:C
- removed D1: D_TVS, Diode_SMD:D_SMB_Handsoldering, symbol Device:D_TVS
- removed D2: SS34, Diode_SMD:D_SMB_Handsoldering, symbol Device:D_Schottky
- removed R1: 100k, Resistor_SMD:R_0805_2012Metric_Pad1.20x1.40mm_HandSolder, symbol Device:R
- removed R2: 20k, Resistor_SMD:R_0805_2012Metric_Pad1.20x1.40mm_HandSolder, symbol Device:R
- removed U1: MP2359DJ-LF-Z, Package_TO_SOT_SMD:TSOT-23-6_HandSoldering, symbol MP2359DJ-LF-Z:MP2359DJ-LF-Z
- added D1: SS34, Diode_SMD:D_SMB_Handsoldering, symbol Device:D
- added D19: LED, LED_SMD:LED_2010_5025Metric_Pad1.52x2.65mm_HandSolder, symbol Device:LED
- added R4: 1K, Resistor_SMD:R_0805_2012Metric_Pad1.20x1.40mm_HandSolder, symbol Device:R
- added U1: AP63205WU-7, Package_TO_SOT_SMD:TSOT-23-6, symbol Regulator_Switching:AP63205WU
- C3, C4: value 22uF 10V -> 22µF
- C5: value 10uF -> 10µF
- C6: value 10uF -> 22µF
- L1: value 22uH -> 4.7µH; footprint Inductor_SMD:L_Bourns_SRR1260 -> Inductor_SMD:L_7.3x7.3_H4.5
Connections:
- net +3.3V: now also D1.2 (A), D19.2 (A)
- net +5V: now also D1.1 (K), U1.1 (FB)
- net +BATT: now also U1.2 (EN), U1.3 (IN)
- net at C2.2, L1.1: now also U1.6 (BST)
- net at C2.1: now also U1.5 (SW)
- net -BATT renamed GND
- net GND: now also R4.2, U1.4 (GND)
- new net: D19.1 (K), R4.1
Other:
- removed sheet Discharge/LED
- removed sheet Fan
- removed sheet LED_Driver
- removed sheet USB-C
- added sheet node1 (node.kicad_sch)
- added sheet node2 (node.kicad_sch)
- added sheet node3 (node.kicad_sch)
- added sheet node4 (node.kicad_sch)
- added sheet node5 (node.kicad_sch)
- moved on the sheet: C1, U2
