File: STM32.kicad_sch (KiCad schematic)
At the start: 16 parts, among them J3 SWD, SW1 BOOT0_BTN, U3 STM32F103C8Tx, Y1 8MHz

Commit message: Complete board redesign
Parts:
- removed C16: 20pF, Capacitor_SMD:C_0805_2012Metric_Pad1.18x1.45mm_HandSolder, symbol Device:C
- removed J3: SWD, Connector_PinHeader_2.54mm:PinHeader_1x04_P2.54mm_Vertical, symbol Connector:Conn_01x04_Socket
- removed R4: 10k, Resistor_SMD:R_0805_2012Metric_Pad1.20x1.40mm_HandSolder, symbol Device:R
- removed R5: 1M, Resistor_SMD:R_0805_2012Metric_Pad1.20x1.40mm_HandSolder, symbol Device:R
- removed Y1: 8MHz, Crystal:Crystal_SMD_3225-4Pin_3.2x2.5mm_HandSoldering, symbol Device:Crystal
- added C25: 10p, Capacitor_SMD:C_0402_1005Metric, symbol Device:C
- added C7: 10u, Capacitor_SMD:C_0603_1608Metric, symbol Device:C
- added C8: 100n, Capacitor_SMD:C_0402_1005Metric, symbol Device:C
- added D13: 1N4148, Diode_THT:D_DO-35_SOD27_P7.62mm_Horizontal, symbol Device:D
- added FB1: 120R, Inductor_SMD:L_0603_1608Metric, symbol Device:FerriteBead
- added J1, J11, J3: Conn_01x04_Male, Connector_PinHeader_2.00mm:PinHeader_1x04_P2.00mm_Vertical, symbol Connector:Conn_01x04_Male
- added J2: USB_C_Receptacle_USB2.0_16P, Connector_USB:USB_C_Receptacle_HRO_TYPE-C-31-M-12, symbol Connector:USB_C_Receptacle_USB2.0_16P
- added J9: FAN, Connector_PinHeader_2.54mm:PinHeader_1x02_P2.54mm_Vertical, symbol Connector:Conn_01x02_Socket
- added Q6: 2N2222, Package_TO_SOT_THT:TO-92_Inline, symbol Transistor_BJT:Q_NPN_BCE
- added R2: 10k, Resistor_SMD:R_0402_1005Metric, symbol Device:R
- added R54: 100, Resistor_SMD:R_0805_2012Metric_Pad1.20x1.40mm_HandSolder, symbol Device:R
- added RP_SCL1, RP_SDA1: 2k2, Resistor_SMD:R_0402_1005Metric, symbol Device:R
- added Y1: 16MHz, Crystal:Crystal_SMD_3225-4Pin_3.2x2.5mm, symbol Device:Crystal_GND24
- C10, C11, C12, C9: value 100nF -> 100n; footprint Capacitor_SMD:C_0805_2012Metric_Pad1.18x1.45mm_HandSolder -> Capacitor_SMD:C_0402_1005Metric
- C13: value 1uF -> 10n; footprint Capacitor_SMD:C_0805_2012Metric_Pad1.18x1.45mm_HandSolder -> Capacitor_SMD:C_0402_1005Metric
- C14: value 10nF -> 1u; footprint Capacitor_SMD:C_0805_2012Metric_Pad1.18x1.45mm_HandSolder -> Capacitor_SMD:C_0402_1005Metric
- C15: value 100nF -> 1u; footprint Capacitor_SMD:C_0805_2012Metric_Pad1.18x1.45mm_HandSolder -> Capacitor_SMD:C_0402_1005Metric
- C17: value 20pF -> 10p; footprint Capacitor_SMD:C_0805_2012Metric_Pad1.18x1.45mm_HandSolder -> Capacitor_SMD:C_0402_1005Metric
- R3: value 10k -> 1k5; footprint Resistor_SMD:R_0805_2012Metric_Pad1.20x1.40mm_HandSolder -> Resistor_SMD:R_0402_1005Metric
- SW1: value BOOT0_BTN -> SW_Push
- U3: value STM32F103C8Tx -> STM32F103C8T6
Connections:
- net +3.3V: now also C10.1, C11.1, C12.1, C15.1, C9.1, SW1.1, C7.1, FB1.2, J1.1 (Pin_1), J11.1 (Pin_1), J3.1 (Pin_1), RP_SCL1.1, RP_SDA1.2; no longer C10.2, C11.2, C12.2, C13.2, C14.2, C9.2, SW1.2, U3.9 (VDDA)
- net FAN_CTRL: now also U3.31 (PA10), R54.1; no longer U3.45 (PB8)
- net GATE_P1: now also U3.15 (PA5); no longer U3.18 (PB0)
- net GATE_P2: now also U3.16 (PA6); no longer U3.19 (PB1)
- net GATE_P3: now also U3.17 (PA7); no longer U3.20 (PB2)
- net GATE_P4: now also U3.29 (PA8); no longer U3.39 (PB3)
- net GATE_P5: now also U3.30 (PA9); no longer U3.40 (PB4)
- net SWDIO: now reaches U3.34 (PA13)
- net SWDIO: now also J11.2 (Pin_2)
- net SWCLK: now reaches U3.37 (PA14)
- net SWCLK: now also J11.3 (Pin_3)
- net at U3.44 (BOOT0): now also SW1.2, R2.2; no longer SW1.1
- net HSE_IN: now reaches U3.5 (PD0)
- net HSE_IN: now also C17.1, Y1.1
- net HSE_OUT: now reaches U3.6 (PD1)
- net HSE_OUT: now also C25.1, Y1.3; no longer C17.1
- net I2C2_SCL: now reaches U3.21 (PB10)
- net I2C2_SCL: now also J3.2 (Pin_2), RP_SCL1.2
- net I2C2_SDA: now reaches U3.22 (PB11)
- net I2C2_SDA: now also J3.3 (Pin_3), RP_SDA1.1
- removed net -BATT: C10.1, C11.1, C12.1, C13.1, C14.1, C15.1, C17.2, C9.1, U3.23 (VSS), U3.35 (VSS), U3.47 (VSS), U3.8 (VSSA)
- net I2C_SCL renamed USART1_TX
- net USART1_TX: now also J1.2 (Pin_2)
- net I2C_SDA renamed USART1_RX
- net USART1_RX: now also J1.3 (Pin_3)
- net USB_DM renamed USB_D-
- net USB_D-: now also J2.A7 (D-), J2.B7 (D-)
- net USB_DP renamed USB_D+
- net USB_D+: now also R3.2, J2.A6 (D+), J2.B6 (D+)
- new net: Q6.1 (B), R54.2
- new net: D13.1 (K), J9.1 (Pin_1), Q6.2 (C)
- new net: C13.1, C14.1, FB1.1, U3.9 (VDDA)
- new net +5V: D13.2 (A), J2.A4 (VBUS), J2.A9 (VBUS), J2.B4 (VBUS), J2.B9 (VBUS), J9.2 (Pin_2)
- new net GND: C10.2, C11.2, C12.2, C13.2, C14.2, C15.2, C17.2, C25.2, C7.2, C8.2, C9.2, J1.4 (Pin_4), J11.4 (Pin_4), J2.A1 (GND), J2.A12 (GND), J2.B1 (GND), J2.B12 (GND), J3.4 (Pin_4), Q6.3 (E), R2.1, U3.23 (VSS), U3.35 (VSS), U3.47 (VSS), U3.8 (VSSA), Y1.2, Y1.4
- new net NRST: C8.1, U3.7 (NRST)
- no-connect marks 18 -> 21
Other:
- note added: "1x 100uF per VDD"
- note added: "Analog Power Filtering"
- note added: "CL = 2*(CL0-Cs)=2*(10-5)pF=10pF"
- note added: "Decoupled Power"
